File: Mini-Lora/Mini-Lora.kicad_pcb (KiCad board)
At the start: 2 copper layers, 68.8 x 25.7 mm, 18 parts, among them J1 BATT, J2 BATT, U1 RFM95W-915S2

Commit message: More updates before fab
Parts:
- added I2C2: CON_HEADER_1X04'NO_LOCK', Curtis_Items:PinHeader_1x04_P2.54mm_Horizontal_SMD, B.Cu at (179.6, 94.2)
- I2C1: footprint Mini-Lora:1X04_NO_LOCK -> Curtis_Items:PinHeader_1x04_P2.54mm_Horizontal_SMD; moved to B.Cu
- moved I2C1 3.80 mm to (164.4, 115.8), turned to -90 degrees
- moved C2 0.15 mm to (133.7, 94.8)
Routing:
- net +3V3: track 137.3 -> 166.9 mm, vias 2 -> 3
- net GND: track 2.65 -> 14.0 mm, vias 170 -> 205
- net /TX: track 0.00 -> 3.20 mm
- net /RX: track 0.00 -> 3.20 mm
Other:
- board text added: "BLU"
- board text added: "BTN"
- board text added: "DIO0"
- board text added: "DIO5"
- board text added: "GRN"
- board text added: "Mini-Lora-NRF52"
- board text added: "Mini-Lora-NRF52 V1.1a"
- board text added: "RED"
- board text added: "uRST"
- board text removed: "A0"
- board text removed: "A1"
- board text removed: "D3"
- board text removed: "D4"
- board text removed: "D5"
- board text removed: "D5 B"
- board text removed: "D6"
- board text removed: "D6 G"
- board text removed: "D9"
- board text removed: "D9 R"
- board text removed: "Mini-Lora"
- board text removed: "Mini-Lora V1.1a"
- board text removed: "V1.1a"
