File: Mini-Lora/Mini-Lora.kicad_sch (KiCad schematic)
At the start: 18 parts, among them J1 BATT, J2 BATT, U1 RFM95W-915S2

Commit message: More updates before fab
Parts:
- added I2C2: CON_HEADER_1X04'NO_LOCK', Curtis_Items:PinHeader_1x04_P2.54mm_Horizontal_SMD, symbol Mini-Lora-eagle-import:CON_HEADER_1X04'NO_LOCK'
- I2C1: footprint Mini-Lora:1X04_NO_LOCK -> Curtis_Items:PinHeader_1x04_P2.54mm_Horizontal_SMD
Connections:
- net +3V3: now also I2C2.1
- net GND: now also I2C2.4
- net RX: now also I2C2.3
- net TX: now also I2C2.2
Changed lines of the file:
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@@
 	(paper "User" 318.77 224.942)
 	(junction
-		(at 59.69 130.81)
-		(diameter 0)
-		(color 0 0 0 0)
-	)
-	(junction
 		(at 26.924 15.367)
 		(diameter 0)
@@
 	)
 	(junction
+		(at 150.368 124.46)
+		(diameter 0)
+		(color 0 0 0 0)
+	)
+	(junction
 		(at 26.924 27.051)
 		(diameter 0)
@@
 	)
 	(junction
-		(at 93.98 71.12)
+		(at 59.69 130.81)
 		(diameter 0)
 		(color 0 0 0 0)
 	)
 	(junction
-		(at 162.56 129.286)
+		(at 93.98 71.12)
 		(diameter 0)
 		(color 0 0 0 0)
 	)
 	(junction
-		(at 162.56 114.935)
+		(at 162.56 129.286)
 		(diameter 0)
 		(color 0 0 0 0)
 	)
 	(junction
-		(at 63.5 115.57)
+		(at 162.56 114.3)
 		(diameter 0)
 		(color 0 0 0 0)
 	)
 	(junction
-		(at 153.67 124.46)
+		(at 63.5 115.57)
 		(diameter 0)
 		(color 0 0 0 0)
@@
 	(wire
 		(pts
-			(xy 162.56 129.286) (xy 171.45 129.286)
+			(xy 162.56 129.286) (xy 173.863 129.286)
+		)
+		(stroke
+			(width 0.1524)
+			(type solid)
+		)
+	)
+	(wire
+		(pts
+			(xy 173.863 119.38) (xy 171.45 119.38)
 		)
 		(stroke
@@
 	(wire
 		(pts
-			(xy 162.56 114.935) (xy 171.45 114.935)
+			(xy 162.56 114.3) (xy 173.863 114.3)
 		)
 		(stroke
@@
 	(wire
 		(pts
-			(xy 162.56 114.935) (xy 153.67 114.935)
+			(xy 162.56 114.3) (xy 150.368 114.3)
 		)
 		(stroke
@@
 	(wire
 		(pts
-			(xy 171.45 114.935) (xy 171.45 119.38)
+			(xy 173.863 114.3) (xy 173.863 119.38)
 		)
 		(stroke
@@
 	(wire
 		(pts
-			(xy 153.67 119.38) (xy 153.67 114.935)
+			(xy 150.368 119.38) (xy 150.368 114.3)
 		)
 		(stroke
@@
 	(wire
 		(pts
-			(xy 153.67 124.46) (xy 153.67 129.286)
+			(xy 150.368 124.46) (xy 150.368 129.286)
 		)
 		(stroke
@@
 	(wire
 		(pts
+			(xy 150.368 119.38) (xy 153.67 119.38)
+		)
+		(stroke
+			(width 0.1524)
+			(type solid)
+		)
+	)
+	(wire
+		(pts
+			(xy 98.044 116.332) (xy 102.235 116.332)
+		)
+		(stroke
+			(width 0)
+			(type default)
+		)
+	)
+	(wire
+		(pts
 			(xy 159.385 60.325) (xy 167.386 60.325)
 		)
@@
 	(wire
 		(pts
+			(xy 98.044 113.792) (xy 102.235 113.792)
+		)
+		(stroke
+			(width 0)
+			(type default)
+		)
+	)
+	(wire
+		(pts
 			(xy 67.31 118.11) (xy 67.31 115.57)
 		)
@@
 	(wire
 		(pts
+			(xy 150.368 124.46) (xy 153.67 124.46)
+		)
+		(stroke
+			(width 0.1524)
+			(type solid)
+		)
+	)
+	(wire
+		(pts
 			(xy 35.687 22.479) (xy 41.021 22.479)
 		)
@@
 	(wire
 		(pts
+			(xy 59.69 130.81) (xy 82.55 130.81)
+		)
+		(stroke
+			(width 0)
+			(type default)
+		)
+	)
+	(wire
+		(pts
 			(xy 132.08 85.725) (xy 144.145 85.725)
 		)
@@
 	(wire
 		(pts
+			(xy 173.863 124.46) (xy 171.45 124.46)
+		)
+		(stroke
+			(width 0.1524)
+			(type solid)
+		)
+	)
+	(wire
+		(pts
 			(xy 97.155 71.12) (xy 93.98 71.12)
 		)
@@
 	(wire
 		(pts
+			(xy 98.044 118.872) (xy 102.235 118.872)
+		)
+		(stroke
+			(width 0)
+			(type default)
+		)
+	)
+	(wire
+		(pts
 			(xy 190.246 60.325) (xy 197.485 60.325)
 		)
@@
 	(wire
 		(pts
-			(xy 153.67 129.286) (xy 162.56 129.286)
+			(xy 150.368 129.286) (xy 162.56 129.286)
 		)
 		(stroke
@@
 	(wire
 		(pts
-			(xy 82.55 130.81) (xy 62.23 130.81)
+			(xy 98.044 121.412) (xy 102.235 121.412)
 		)
 		(stroke
@@
 	(wire
 		(pts
-			(xy 59.69 130.81) (xy 82.55 130.81)
-		)
-		(stroke
-			(width 0.1524)
-			(type solid)
-		)
-	)
-	(wire
-		(pts
 			(xy 63.5 113.03) (xy 63.5 115.57)
 		)
@@
 	(wire
 		(pts
-			(xy 162.56 114.935) (xy 162.56 111.633)
+			(xy 162.56 114.3) (xy 162.56 110.998)
 		)
 		(stroke
@@
 	(wire
 		(pts
-			(xy 144.78 124.46) (xy 153.67 124.46)
+			(xy 144.78 124.46) (xy 150.368 124.46)
 		)
 		(stroke
@@
 	(wire
 		(pts
-			(xy 171.45 129.286) (xy 171.45 124.46)
+			(xy 173.863 129.286) (xy 173.863 124.46)
 		)
 		(stroke
@@
 		)
 	)
+	(label "TX"
+		(at 102.235 116.332 180)
+		(fields_autoplaced yes)
+		(effects
+			(font
+				(size 1.27 1.27)
+			)
+			(justify right bottom)
+		)
+	)
 	(label "SS"
 		(at 81.28 83.82 180)
@@
 		)
 	)
+	(label "GND"
+		(at 102.235 121.412 180)
+		(fields_autoplaced yes)
+		(effects
+			(font
+				(size 1.27 1.27)
+			)
+			(justify right bottom)
+		)
+	)
 	(label "A2"
 		(at 190.246 70.485 0)
@@
 		)
 	)
+	(label "RX"
+		(at 102.235 118.872 180)
+		(fields_autoplaced yes)
+		(effects
+			(font
+				(size 1.27 1.27)
+			)
+			(justify right bottom)
+		)
+	)
 	(label "SCL"
 		(at 53.34 133.35 0)
@@
 	)
 	(label "3V3"
-		(at 153.67 119.38 0)
+		(at 150.368 119.38 0)
 		(fields_autoplaced yes)
 		(effects
@@
 		)
 	)
+	(label "3V3"
+		(at 102.235 113.792 180)
+		(fields_autoplaced yes)
+		(effects
+			(font
+				(size 1.27 1.27)
+			)
+			(justify right bottom)
+		)
+	)
 	(label "BAT+"
 		(at 190.246 55.245 0)
@@
 	)
 	(symbol
+		(lib_id "Mini-Lora-eagle-import:CON_HEADER_1X04'NO_LOCK'")
+		(at 112.395 111.252 180)
+		(unit 1)
+		(exclude_from_sim no)
+		(in_bom yes)
+		(on_board yes)
+		(dnp no)
+		(property "Reference" "I2C2"
+			(at 110.236 124.968 0)
+			(effects
+				(font
+					(size 1.778 1.5113)
+				)
+				(justify left bottom)
+			)
+		)
+		(property "Value" "CON_HEADER_1X04'NO_LOCK'"
+			(at 111.125 108.712 0)
+			(effects
+				(font
+					(size 1.778 1.5113)
+				)
+				(justify left bottom)
+				(hide yes)
+			)
+		)
+		(property "Footprint" "Curtis_Items:PinHeader_1x04_P2.54mm_Horizontal_SMD"
+			(at 112.395 111.252 0)
+			(effects
+				(font
+					(size 1.27 1.27)
+				)
+				(hide yes)
+			)
+		)
+		(property "Datasheet" ""
+			(at 112.395 111.252 0)
+			(effects
+				(font
+					(size 1.27 1.27)
+				)
+				(hide yes)
+			)
+		)
+		(property "Description" ""
+			(at 112.395 111.252 0)
+			(effects
+				(font
+					(size 1.27 1.27)
+				)
+				(hide yes)
+			)
+		)
+		(pin "1"
+		)
+		(pin "3"
+		)
+		(pin "2"
+		)
+		(pin "4"
+		)
+		(instances
+			(project "Mini-Lora"
+				(path "/774ec7ed-5802-4160-ad3c-1080ce78b57b"
+					(reference "I2C2")
+					(unit 1)
+				)
+			)
+		)
+	)
+	(symbol
 		(lib_id "power:+BATT")
 		(at 26.924 14.351 0)
@@
 			)
 		)
-		(property "Footprint" "Mini-Lora:1X04_NO_LOCK"
+		(property "Footprint" "Curtis_Items:PinHeader_1x04_P2.54mm_Horizontal_SMD"
 			(at 92.71 124.333 0)
 			(effects
@@
 		(dnp no)
 		(property "Reference" "BTN0"
-			(at 157.48 116.84 0)
+			(at 157.226 116.586 0)
 			(effects
 				(font
@@
 		)
 		(property "Value" "DHT-4235A"
-			(at 157.48 128.27 0)
+			(at 157.734 128.778 0)
 			(effects
 				(font
@@
 	(symbol
 		(lib_id "Mini-Lora-eagle-import:+3V3")
-		(at 162.56 109.093 0)
+		(at 162.56 108.458 0)
 		(unit 1)
 		(exclude_from_sim no)
@@
 		(dnp no)
 		(property "Reference" "#+3V02"
-			(at 162.56 109.093 0)
+			(at 162.56 108.458 0)
 			(effects
 				(font
@@
 		)
 		(property "Value" "3V3"
-			(at 165.1 106.553 90)
+			(at 165.1 105.918 90)
 			(effects
 				(font
@@
 		)
 		(property "Footprint" ""
-			(at 162.56 109.093 0)
+			(at 162.56 108.458 0)
 			(effects
 				(font
@@
 		)
 		(property "Datasheet" ""
-			(at 162.56 109.093 0)
+			(at 162.56 108.458 0)
 			(effects
 				(font
@@
 		)
 		(property "Description" ""
-			(at 162.56 109.093 0)
+			(at 162.56 108.458 0)
 			(effects
 				(font
